Commit message: 6_17日看代码的时候随便写了几行注释

File: src/moveit_resources-ros2/dual_arm_jaka_c5_moveit_config/config/jaka_c5_arm_macro.xacro (robot description, xacro)
@@ -13,9 +13,14 @@
     <!-- Link_00 (base) -->
     <link name="${prefix}Link_00">
-      <inertial>
+      <!-- 惯性参数 -->
+      <inertial>
+        <!-- 重心位置 -->
         <origin xyz="0.0028167 -0.00019454 0.019544" rpy="0 0 0" />
+        <!-- 质量(0.5公斤) -->
         <mass value="0.52663" />
+        <!-- 转动惯量矩阵 -->
         <inertia ixx="0.0006297" ixy="6.7091E-08" ixz="3.4682E-06" iyy="0.00095727" iyz="2.4476E-07" izz="0.0014514" />
       </inertial>
+      <!-- 可视化外观 -->
       <visual>
         <origin xyz="0 0 0" rpy="0 0 0" />
@@ -27,4 +32,5 @@
         </material>
       </visual>
+      <!-- 碰撞模型 物理安全的"骨架" -->
       <collision>
         <origin xyz="0 0 0" rpy="0 0 0" />
@@ -58,8 +64,13 @@
     </link>
     <joint name="${prefix}joint_1" type="revolute">
+      <!-- 子坐标相对于父坐标的偏移 -->
       <origin xyz="0 -0.00022535 0.12015" rpy="0 0 0" />
+      <!-- 定义父级 -->
       <parent link="${prefix}Link_00" />
+      <!-- 定义子级 -->
       <child link="${prefix}Link_01" />
-      <axis xyz="0 0 1" />
+      <!-- 定义旋转轴 关节的运动方向 -->
+      <axis xyz="0 0 1" />
+       <!-- 软件限位 -->
       <limit lower="-6.28" upper="6.28" effort="2000" velocity="3.14" />
     </joint>

Commit message: 初步修改了人模型和机械臂的放置位置 但是机械臂和床穿模了 床还是浮空不合理 机械臂的按摩运动不动了

File: src/moveit_resources-ros2/dual_arm_jaka_c5_moveit_config/config/jaka_c5_arm_macro.xacro (robot description, xacro)
@@ -1,5 +1,5 @@
 <?xml version="1.0" ?>
 <robot xmlns:xacro="http://www.ros.org/wiki/xacro">
-  <xacro:macro name="jaka_c5_arm" params="name prefix parent *origin initial_positions_file hardware_plugin grip_pad_contact_z grip_pad_inward_sign">
+  <xacro:macro name="jaka_c5_arm" params="name prefix parent *origin initial_positions_file hardware_plugin grip_pad_contact_z grip_pad_inward_sign use_flange">
     <!-- ros2_control -->
     <xacro:include filename="$(find dual_arm_jaka_c5_moveit_config)/config/jaka_c5.ros2_control.xacro" />
@@ -226,42 +226,45 @@
     </joint>
     <!-- Flat passive clamp pad used by the carry demo. The contact frame sits on
-         the pad face that should touch the box side. -->
-    <xacro:property name="grip_pad_thickness" value="0.012"/>
-    <xacro:property name="grip_pad_width" value="0.085"/>
-    <xacro:property name="grip_pad_height" value="0.085"/>
-    <xacro:property name="grip_pad_center_z" value="${grip_pad_contact_z - grip_pad_inward_sign * grip_pad_thickness / 2.0}"/>
-    <link name="${prefix}grip_pad">
-      <inertial>
-        <origin xyz="0 0 0" rpy="0 0 0" />
-        <mass value="0.05" />
-        <inertia ixx="0.00008" ixy="0" ixz="0" iyy="0.00008" iyz="0" izz="0.00008" />
-      </inertial>
-      <visual>
-        <origin xyz="0 0 0" rpy="0 0 0" />
-        <geometry>
-          <box size="${grip_pad_width} ${grip_pad_height} ${grip_pad_thickness}" />
-        </geometry>
-        <material name="${prefix}grip_pad_material">
-          <color rgba="0.06 0.08 0.09 1.0" />
-        </material>
-      </visual>
-      <collision>
-        <origin xyz="0 0 0" rpy="0 0 0" />
-        <geometry>
-          <box size="${grip_pad_width} ${grip_pad_height} ${grip_pad_thickness}" />
-        </geometry>
-      </collision>
-    </link>
-    <joint name="${prefix}grip_pad_joint" type="fixed">
-      <origin xyz="0 0 ${grip_pad_center_z}" rpy="0 0 0" />
-      <parent link="${prefix}Link_06" />
-      <child link="${prefix}grip_pad" />
-    </joint>
-    <link name="${prefix}grip_contact"/>
-    <joint name="${prefix}grip_contact_joint" type="fixed">
-      <origin xyz="0 0 ${grip_pad_contact_z}" rpy="0 0 0" />
-      <parent link="${prefix}Link_06" />
-      <child link="${prefix}grip_contact" />
-    </joint>
+         the pad face that should touch the box side.
+         条件包含：use_flange=false（按摩Demo）时跳过，避免末端法兰影响按摩。 -->
+    <xacro:if value="${use_flange}">
+      <xacro:property name="grip_pad_thickness" value="0.012"/>
+      <xacro:property name="grip_pad_width" value="0.085"/>
+      <xacro:property name="grip_pad_height" value="0.085"/>
+      <xacro:property name="grip_pad_center_z" value="${grip_pad_contact_z - grip_pad_inward_sign * grip_pad_thickness / 2.0}"/>
+      <link name="${prefix}grip_pad">
+        <inertial>
+          <origin xyz="0 0 0" rpy="0 0 0" />
+          <mass value="0.05" />
+          <inertia ixx="0.00008" ixy="0" ixz="0" iyy="0.00008" iyz="0" izz="0.00008" />
+        </inertial>
+        <visual>
+          <origin xyz="0 0 0" rpy="0 0 0" />
+          <geometry>
+            <box size="${grip_pad_width} ${grip_pad_height} ${grip_pad_thickness}" />
+          </geometry>
+          <material name="${prefix}grip_pad_material">
+            <color rgba="0.06 0.08 0.09 1.0" />
+          </material>
+        </visual>
+        <collision>
+          <origin xyz="0 0 0" rpy="0 0 0" />
+          <geometry>
+            <box size="${grip_pad_width} ${grip_pad_height} ${grip_pad_thickness}" />
+          </geometry>
+        </collision>
+      </link>
+      <joint name="${prefix}grip_pad_joint" type="fixed">
+        <origin xyz="0 0 ${grip_pad_center_z}" rpy="0 0 0" />
+        <parent link="${prefix}Link_06" />
+        <child link="${prefix}grip_pad" />
+      </joint>
+      <link name="${prefix}grip_contact"/>
+      <joint name="${prefix}grip_contact_joint" type="fixed">
+        <origin xyz="0 0 ${grip_pad_contact_z}" rpy="0 0 0" />
+        <parent link="${prefix}Link_06" />
+        <child link="${prefix}grip_contact" />
+      </joint>
+    </xacro:if>
   </xacro:macro>
 </robot>

File: src/moveit_resources-ros2/dual_arm_jaka_c5_moveit_config/config/jaka_c5_dual.urdf.xacro (robot description, xacro)
@@ -7,9 +7,14 @@
   <xacro:arg name="hardware_plugin" default="mock_components/GenericSystem"/>
   <xacro:arg name="use_gazebo" default="false"/>
+  <xacro:arg name="use_flange" default="true"/>
+  <xacro:arg name="left_arm_x" default="0"/>
+  <xacro:arg name="left_arm_y" default="-0.25"/>
+  <xacro:arg name="right_arm_x" default="0"/>
+  <xacro:arg name="right_arm_y" default="0.25"/>
   <!-- Root link -->
   <link name="world"/>
   <!-- Xacro imports -->
   <xacro:include filename="jaka_c5_arm_macro.xacro" />
-  <!-- Left arm: placed -0.25m along Y axis -->
+  <!-- Left arm: 位置由 launch 文件通过 xacro:arg 控制 -->
   <xacro:jaka_c5_arm
       name="left_jaka_c5"
@@ -19,8 +24,9 @@
       grip_pad_contact_z="0.012"
       grip_pad_inward_sign="1"
-      initial_positions_file="$(arg left_initial_positions_file)">
-      <origin xyz="0 -0.25 0" rpy="0 0 0" />
+      initial_positions_file="$(arg left_initial_positions_file)"
+      use_flange="$(arg use_flange)">
+      <origin xyz="$(arg left_arm_x) $(arg left_arm_y) 0" rpy="0 0 0" />
   </xacro:jaka_c5_arm>
-  <!-- Right arm: placed +0.25m along Y axis -->
+  <!-- Right arm: 位置由 launch 文件通过 xacro:arg 控制 -->
   <xacro:jaka_c5_arm
       name="right_jaka_c5"
@@ -30,6 +36,7 @@
       grip_pad_contact_z="0.012"
       grip_pad_inward_sign="1"
-      initial_positions_file="$(arg right_initial_positions_file)">
-      <origin xyz="0 0.25 0" rpy="0 0 0" />
+      initial_positions_file="$(arg right_initial_positions_file)"
+      use_flange="$(arg use_flange)">
+      <origin xyz="$(arg right_arm_x) $(arg right_arm_y) 0" rpy="0 0 0" />
   </xacro:jaka_c5_arm>
   <xacro:if value="$(arg use_gazebo)">

Commit message: 机械臂可以动了 但是运动一会后就开始抽风了 rviz里面人模型的上半背部会陷进床里面 但是gazebo 是正常的  gazebo和rviz程序的启动好慢

File: src/moveit_resources-ros2/dual_arm_jaka_c5_moveit_config/config/jaka_c5_arm_macro.xacro (robot description, xacro)
@@ -74,4 +74,5 @@
        <!-- 软件限位 -->
       <limit lower="-6.28" upper="6.28" effort="2000" velocity="3.14" />
+      <dynamics damping="2.0" friction="0.20" />
     </joint>
     <!-- Joint_2: Link_01 -> Link_02 -->
@@ -104,4 +105,5 @@
       <axis xyz="0 0 1" />
       <limit lower="-1.48" upper="4.62" effort="5000" velocity="3.14" />
+      <dynamics damping="8.0" friction="0.30" />
     </joint>
     <!-- Joint_3: Link_02 -> Link_03 -->
@@ -134,4 +136,5 @@
       <axis xyz="0 0 1" />
       <limit lower="-3.05" upper="3.05" effort="5000" velocity="3.14" />
+      <dynamics damping="6.0" friction="0.25" />
     </joint>
     <!-- Joint_4: Link_03 -> Link_04 -->
@@ -164,4 +167,5 @@
       <axis xyz="0 0 1" />
       <limit lower="-1.48" upper="4.62" effort="2000" velocity="3.14" />
+      <dynamics damping="4.0" friction="0.20" />
     </joint>
     <!-- Joint_5: Link_04 -> Link_05 -->
@@ -194,4 +198,5 @@
       <axis xyz="0 0 1" />
       <limit lower="-6.28" upper="6.28" effort="3000" velocity="3.14" />
+      <dynamics damping="2.0" friction="0.15" />
     </joint>
     <!-- Joint_6: Link_05 -> Link_06 (end effector mount) -->
@@ -224,5 +229,14 @@
       <axis xyz="0 0 1" />
       <limit lower="-6.28" upper="6.28" effort="1000" velocity="3.14" />
-    </joint>
+      <dynamics damping="1.0" friction="0.10" />
+    </joint>
+    <xacro:if value="$(arg use_gazebo)">
+      <gazebo reference="${prefix}joint_1"><implicitSpringDamper>true</implicitSpringDamper></gazebo>
+      <gazebo reference="${prefix}joint_2"><implicitSpringDamper>true</implicitSpringDamper></gazebo>
+      <gazebo reference="${prefix}joint_3"><implicitSpringDamper>true</implicitSpringDamper></gazebo>
+      <gazebo reference="${prefix}joint_4"><implicitSpringDamper>true</implicitSpringDamper></gazebo>
+      <gazebo reference="${prefix}joint_5"><implicitSpringDamper>true</implicitSpringDamper></gazebo>
+      <gazebo reference="${prefix}joint_6"><implicitSpringDamper>true</implicitSpringDamper></gazebo>
+    </xacro:if>
     <!-- Flat passive clamp pad used by the carry demo. The contact frame sits on
          the pad face that should touch the box side.
