Commit message: jakac5双臂协同搬运物体到桌面

File: src/moveit_resources-ros2/dual_arm_jaka_c5_moveit_config/config/jaka_c5.ros2_control.xacro (robot description, xacro)
@@ -1,9 +1,9 @@
 <?xml version="1.0"?>
 <robot xmlns:xacro="http://www.ros.org/wiki/xacro">
-  <xacro:macro name="jaka_c5_arm_ros2_control" params="name initial_positions_file prefix">
+  <xacro:macro name="jaka_c5_arm_ros2_control" params="name initial_positions_file prefix hardware_plugin">
     <xacro:property name="initial_positions" value="${xacro.load_yaml(initial_positions_file)['initial_positions']}"/>
     <ros2_control name="${prefix}${name}" type="system">
       <hardware>
-        <plugin>mock_components/GenericSystem</plugin>
+        <plugin>${hardware_plugin}</plugin>
       </hardware>
       <joint name="${prefix}joint_1">

File: src/moveit_resources-ros2/dual_arm_jaka_c5_moveit_config/config/jaka_c5_arm_macro.xacro (robot description, xacro)
@@ -1,8 +1,8 @@
 <?xml version="1.0" ?>
 <robot xmlns:xacro="http://www.ros.org/wiki/xacro">
-  <xacro:macro name="jaka_c5_arm" params="name prefix parent *origin initial_positions_file">
+  <xacro:macro name="jaka_c5_arm" params="name prefix parent *origin initial_positions_file hardware_plugin grip_pad_contact_z grip_pad_inward_sign">
     <!-- ros2_control -->
     <xacro:include filename="$(find dual_arm_jaka_c5_moveit_config)/config/jaka_c5.ros2_control.xacro" />
-    <xacro:jaka_c5_arm_ros2_control name="${name}" initial_positions_file="${initial_positions_file}" prefix="${prefix}"/>
+    <xacro:jaka_c5_arm_ros2_control name="${name}" initial_positions_file="${initial_positions_file}" prefix="${prefix}" hardware_plugin="${hardware_plugin}"/>
     <!-- base_joint fixes the arm base to the environment (world) -->
     <joint name="${prefix}base_joint" type="fixed">
@@ -225,4 +225,43 @@
       <limit lower="-6.28" upper="6.28" effort="1000" velocity="3.14" />
     </joint>
+    <!-- Flat passive clamp pad used by the carry demo. The contact frame sits on
+         the pad face that should touch the box side. -->
+    <xacro:property name="grip_pad_thickness" value="0.012"/>
+    <xacro:property name="grip_pad_width" value="0.085"/>
+    <xacro:property name="grip_pad_height" value="0.085"/>
+    <xacro:property name="grip_pad_center_z" value="${grip_pad_contact_z - grip_pad_inward_sign * grip_pad_thickness / 2.0}"/>
+    <link name="${prefix}grip_pad">
+      <inertial>
+        <origin xyz="0 0 0" rpy="0 0 0" />
+        <mass value="0.05" />
+        <inertia ixx="0.00008" ixy="0" ixz="0" iyy="0.00008" iyz="0" izz="0.00008" />
+      </inertial>
+      <visual>
+        <origin xyz="0 0 0" rpy="0 0 0" />
+        <geometry>
+          <box size="${grip_pad_width} ${grip_pad_height} ${grip_pad_thickness}" />
+        </geometry>
+        <material name="${prefix}grip_pad_material">
+          <color rgba="0.06 0.08 0.09 1.0" />
+        </material>
+      </visual>
+      <collision>
+        <origin xyz="0 0 0" rpy="0 0 0" />
+        <geometry>
+          <box size="${grip_pad_width} ${grip_pad_height} ${grip_pad_thickness}" />
+        </geometry>
+      </collision>
+    </link>
+    <joint name="${prefix}grip_pad_joint" type="fixed">
+      <origin xyz="0 0 ${grip_pad_center_z}" rpy="0 0 0" />
+      <parent link="${prefix}Link_06" />
+      <child link="${prefix}grip_pad" />
+    </joint>
+    <link name="${prefix}grip_contact"/>
+    <joint name="${prefix}grip_contact_joint" type="fixed">
+      <origin xyz="0 0 ${grip_pad_contact_z}" rpy="0 0 0" />
+      <parent link="${prefix}Link_06" />
+      <child link="${prefix}grip_contact" />
+    </joint>
   </xacro:macro>
 </robot>

File: src/moveit_resources-ros2/dual_arm_jaka_c5_moveit_config/config/jaka_c5_dual.urdf.xacro (robot description, xacro)
@@ -5,4 +5,6 @@
   <xacro:arg name="right_initial_positions_file"
           default="$(find dual_arm_jaka_c5_moveit_config)/config/right_initial_positions.yaml"/>
+  <xacro:arg name="hardware_plugin" default="mock_components/GenericSystem"/>
+  <xacro:arg name="use_gazebo" default="false"/>
   <!-- Root link -->
   <link name="world"/>
@@ -14,4 +16,7 @@
       prefix="left_"
       parent="world"
+      hardware_plugin="$(arg hardware_plugin)"
+      grip_pad_contact_z="0.012"
+      grip_pad_inward_sign="1"
       initial_positions_file="$(arg left_initial_positions_file)">
       <origin xyz="0 -0.25 0" rpy="0 0 0" />
@@ -22,6 +27,16 @@
       prefix="right_"
       parent="world"
+      hardware_plugin="$(arg hardware_plugin)"
+      grip_pad_contact_z="0.012"
+      grip_pad_inward_sign="1"
       initial_positions_file="$(arg right_initial_positions_file)">
       <origin xyz="0 0.25 0" rpy="0 0 0" />
   </xacro:jaka_c5_arm>
+  <xacro:if value="$(arg use_gazebo)">
+    <gazebo>
+      <plugin filename="libgazebo_ros2_control.so" name="gazebo_ros2_control">
+        <parameters>$(find dual_arm_jaka_c5_moveit_config)/config/ros2_controllers.yaml</parameters>
+      </plugin>
+    </gazebo>
+  </xacro:if>
 </robot>

Commit message: rvizdemo机械臂会碰撞  但是按摩人左右背部

File: src/moveit_resources-ros2/dual_arm_jaka_c5_moveit_config/config/jaka_c5.ros2_control.xacro (robot description, xacro)
@@ -3,5 +3,5 @@
   <xacro:macro name="jaka_c5_arm_ros2_control" params="name initial_positions_file prefix hardware_plugin">
     <xacro:property name="initial_positions" value="${xacro.load_yaml(initial_positions_file)['initial_positions']}"/>
-    <ros2_control name="${prefix}${name}" type="system">
+    <ros2_control name="${name}" type="system">
       <hardware>
         <plugin>${hardware_plugin}</plugin>

File: src/moveit_resources-ros2/dual_arm_jaka_c5_moveit_config/config/jaka_c5_arm_macro.xacro (robot description, xacro)
@@ -229,13 +229,37 @@
       <axis xyz="0 0 1" />
       <limit lower="-6.28" upper="6.28" effort="1000" velocity="3.14" />
-      <dynamics damping="1.0" friction="0.10" />
+      <dynamics damping="15.0" friction="0.20" />
     </joint>
     <xacro:if value="$(arg use_gazebo)">
-      <gazebo reference="${prefix}joint_1"><implicitSpringDamper>true</implicitSpringDamper></gazebo>
-      <gazebo reference="${prefix}joint_2"><implicitSpringDamper>true</implicitSpringDamper></gazebo>
-      <gazebo reference="${prefix}joint_3"><implicitSpringDamper>true</implicitSpringDamper></gazebo>
-      <gazebo reference="${prefix}joint_4"><implicitSpringDamper>true</implicitSpringDamper></gazebo>
-      <gazebo reference="${prefix}joint_5"><implicitSpringDamper>true</implicitSpringDamper></gazebo>
-      <gazebo reference="${prefix}joint_6"><implicitSpringDamper>true</implicitSpringDamper></gazebo>
+      <gazebo reference="${prefix}joint_1">
+        <implicitSpringDamper>true</implicitSpringDamper>
+        <pid>50.0 0.0 3.0</pid>
+        <maxEffort>2.0</maxEffort>
+      </gazebo>
+      <gazebo reference="${prefix}joint_2">
+        <implicitSpringDamper>true</implicitSpringDamper>
+        <pid>50.0 0.0 3.0</pid>
+        <maxEffort>2.0</maxEffort>
+      </gazebo>
+      <gazebo reference="${prefix}joint_3">
+        <implicitSpringDamper>true</implicitSpringDamper>
+        <pid>50.0 0.0 3.0</pid>
+        <maxEffort>2.0</maxEffort>
+      </gazebo>
+      <gazebo reference="${prefix}joint_4">
+        <implicitSpringDamper>true</implicitSpringDamper>
+        <pid>50.0 0.0 3.0</pid>
+        <maxEffort>2.0</maxEffort>
+      </gazebo>
+      <gazebo reference="${prefix}joint_5">
+        <implicitSpringDamper>true</implicitSpringDamper>
+        <pid>50.0 0.0 3.0</pid>
+        <maxEffort>2.0</maxEffort>
+      </gazebo>
+      <gazebo reference="${prefix}joint_6">
+        <implicitSpringDamper>true</implicitSpringDamper>
+        <pid>50.0 0.0 3.0</pid>
+        <maxEffort>2.0</maxEffort>
+      </gazebo>
     </xacro:if>
     <!-- Flat passive clamp pad used by the carry demo. The contact frame sits on
