Commit message: 机械臂仿真替换 图纸转换urdf 水果仿真乱跳修复

File: src/moveit_resources-ros2/single_arm_jaka_c5_pick_place/config/gripper.xacro (robot description, xacro)
@@ -58,5 +58,5 @@
       <child link="left_finger" />
       <axis xyz="0 1 0" />
-      <limit lower="0.0" upper="0.04" effort="50" velocity="0.2" />
+      <limit lower="0.0" upper="0.06" effort="50" velocity="0.2" />
     </joint>
     <!-- Left finger contact frame (tip center for grasp detection) -->
@@ -95,5 +95,5 @@
       <child link="right_finger" />
       <axis xyz="0 1 0" />
-      <limit lower="-0.04" upper="0.0" effort="50" velocity="0.2" />
+      <limit lower="-0.06" upper="0.0" effort="50" velocity="0.2" />
     </joint>
     <!-- Right finger contact frame (tip center for grasp detection) -->

File: src/moveit_resources-ros2/single_arm_jaka_c5_pick_place/config/jaka_c5_pick_place.urdf.xacro (robot description, xacro)
@@ -8,9 +8,9 @@
   <link name="world"/>
   <!-- Xacro imports -->
-  <xacro:include filename="jaka_c5_arm_macro.xacro" />
+  <xacro:include filename="fruit_arm_macro.xacro" />
   <xacro:include filename="gripper.xacro" />
   <xacro:include filename="camera_mount.xacro" />
   <!-- Single arm at world origin -->
-  <xacro:jaka_c5_arm
+  <xacro:fruit_arm
       parent="world"
       hardware_plugin="$(arg hardware_plugin)"
@@ -35,4 +35,34 @@
       </plugin>
     </gazebo>
+    <gazebo>
+      <plugin filename="libfruit_grasp_attach_plugin.so"
+              name="fruit_grasp_attach_plugin">
+        <ros>
+          <namespace>/simulation/fruit_gripper</namespace>
+        </ros>
+        <!-- Gazebo collapses the fixed gripper_base joint into Link_06. -->
+        <parent_link>Link_06</parent_link>
+        <child_link>apple_link</child_link>
+        <model_prefix>fruit_</model_prefix>
+        <!-- Link_06 is 67mm behind tool_flange and the 80mm fingers. -->
+        <max_distance>0.20</max_distance>
+      </plugin>
+    </gazebo>
+    <gazebo reference="left_finger">
+      <mu1>1.2</mu1>
+      <mu2>1.2</mu2>
+      <kp>100000</kp>
+      <kd>10</kd>
+      <maxVel>0.05</maxVel>
+      <minDepth>0.001</minDepth>
+    </gazebo>
+    <gazebo reference="right_finger">
+      <mu1>1.2</mu1>
+      <mu2>1.2</mu2>
+      <kp>100000</kp>
+      <kd>10</kd>
+      <maxVel>0.05</maxVel>
+      <minDepth>0.001</minDepth>
+    </gazebo>
   </xacro:if>
 </robot>
