Commit message: 添加urdf机械限位 和 moveit规划的角度限制

File: src/moveit_resources-ros2/single_arm_jaka_c5_pick_place/config/fruit_arm_macro.xacro (robot description, xacro)
@@ -2,8 +2,8 @@
 <robot xmlns:xacro="http://www.ros.org/wiki/xacro">
   <!--
-    Kinematic model inferred from the supplied STEP assembly.  The drawing pose
-    is q=[0,0,0,0,0,0].  Visual meshes are millimetres and therefore use a
-    0.001 mesh scale.  Collisions are deliberately simple for stable Gazebo and
-    MoveIt performance.
+    Kinematic model inferred from the supplied STEP assembly.  The drawing
+    pose is URDF zero; mechanical reference lines therefore require the
+    documented joint-coordinate offsets below. Visual meshes are millimetres
+    and therefore use a 0.001 mesh scale. Collisions are deliberately simple.
   -->
   <xacro:macro name="fruit_arm" params="parent hardware_plugin initial_positions_file">
@@ -33,5 +33,6 @@
       <parent link="${parent}"/>
       <child link="Link_00"/>
-      <origin xyz="0 0 0" rpy="0 0 0"/>
+      <!-- CAD assembly front is -X; expose mechanical front as world +X. -->
+      <origin xyz="0 0 0" rpy="0 0 3.141592654"/>
     </joint>
     <link name="Link_00">
@@ -56,5 +57,6 @@
       <child link="Link_01"/>
       <axis xyz="0 0 1"/>
-      <limit lower="-3.14" upper="3.14" effort="250" velocity="1.5"/>
+      <!-- Mechanical hard stop: +/-165 deg. -->
+      <limit lower="-2.879793266" upper="2.879793266" effort="250" velocity="1.5"/>
     </joint>
     <link name="Link_02">
@@ -67,9 +69,14 @@
     </link>
     <joint name="joint_2" type="revolute">
-      <origin xyz="-0.048101 0.056781 0.094025" rpy="0 0 0"/>
+      <!-- Re-zero CAD assembly angle -65.196838 deg to mechanical J2=0. -->
+      <origin xyz="-0.048101 0.056781 0.094025" rpy="0 -1.137899491 0"/>
       <parent link="Link_01"/>
       <child link="Link_02"/>
       <axis xyz="0 1 0"/>
-      <limit lower="-2.60" upper="2.60" effort="250" velocity="1.5"/>
+      <!--
+        Positive is clockwise when viewed along +Y. Mechanical hard stops:
+        CCW 60 / CW 80 deg.
+      -->
+      <limit lower="-1.047197551" upper="1.396263402" effort="250" velocity="1.5"/>
     </joint>
     <link name="Link_03">
@@ -82,9 +89,13 @@
     </link>
     <joint name="joint_3" type="revolute">
-      <origin xyz="0.399412 -0.015781 0.184581" rpy="0 0 0"/>
+      <!-- Re-zero CAD assembly angle +57.956279 deg to perpendicular J3=0. -->
+      <origin xyz="0.399412 -0.015781 0.184581" rpy="0 1.011527890 0"/>
       <parent link="Link_02"/>
       <child link="Link_03"/>
       <axis xyz="0 1 0"/>
-      <limit lower="-2.60" upper="2.60" effort="180" velocity="1.5"/>
+      <!--
+        Mechanical hard stop: +/-90 deg from perpendicular upper/forearm.
+      -->
+      <limit lower="-1.570796327" upper="1.570796327" effort="180" velocity="1.5"/>
     </joint>
     <link name="Link_04">
@@ -97,9 +108,11 @@
     </link>
     <joint name="joint_4" type="revolute">
-      <origin xyz="-0.041455 -0.032800 0.057441" rpy="0 0 0"/>
+      <!-- CAD logo-plane reference is opposite mechanical J4 zero. -->
+      <origin xyz="-0.041455 -0.032800 0.057441" rpy="3.141592654 0 0"/>
       <parent link="Link_03"/>
       <child link="Link_04"/>
       <axis xyz="1 0 0"/>
-      <limit lower="-3.14" upper="3.14" effort="120" velocity="1.8"/>
+      <!-- Mechanical hard stop: +/-170 deg. -->
+      <limit lower="-2.967059728" upper="2.967059728" effort="120" velocity="1.8"/>
     </joint>
     <link name="Link_05">
@@ -112,9 +125,13 @@
     </link>
     <joint name="joint_5" type="revolute">
-      <origin xyz="-0.372174 -0.034450 -0.004890" rpy="0 0 0"/>
+      <!-- Re-zero CAD assembly angle +33.439625 deg to mechanical J5=0. -->
+      <origin xyz="-0.372174 -0.034450 -0.004890" rpy="0 0.583631552 0"/>
       <parent link="Link_04"/>
       <child link="Link_05"/>
       <axis xyz="0 1 0"/>
-      <limit lower="-2.60" upper="2.60" effort="100" velocity="1.8"/>
+      <!--
+        Mechanical hard stop: +/-90 deg from the J4-parallel reference.
+      -->
+      <limit lower="-1.570796327" upper="1.570796327" effort="100" velocity="1.8"/>
     </joint>
     <link name="Link_06">
@@ -131,5 +148,6 @@
       <child link="Link_06"/>
       <axis xyz="-0.834467 0 -0.551058"/>
-      <limit lower="-3.14" upper="3.14" effort="80" velocity="2.0"/>
+      <!-- Mechanical hard stop: +/-160 deg. -->
+      <limit lower="-2.792526803" upper="2.792526803" effort="80" velocity="2.0"/>
     </joint>
     <link name="tool_flange"/>

File: src/moveit_resources-ros2/single_arm_jaka_c5_pick_place/config/gripper.xacro (robot description, xacro)
@@ -58,5 +58,6 @@
       <child link="left_finger" />
       <axis xyz="0 1 0" />
-      <limit lower="0.0" upper="0.06" effort="50" velocity="0.2" />
+      <!-- 56mm centre offset gives a 100mm clear inner opening. -->
+      <limit lower="0.0" upper="0.056" effort="50" velocity="0.2" />
     </joint>
     <!-- Left finger contact frame (tip center for grasp detection) -->
@@ -95,5 +96,5 @@
       <child link="right_finger" />
       <axis xyz="0 1 0" />
-      <limit lower="-0.06" upper="0.0" effort="50" velocity="0.2" />
+      <limit lower="-0.056" upper="0.0" effort="50" velocity="0.2" />
     </joint>
     <!-- Right finger contact frame (tip center for grasp detection) -->
