Commit message: Add model joint checks and kinematic calibration support

File: src/moveit_resources-ros2/fruit_arm_moveit_config/config/fruit_arm_macro.xacro (robot description, xacro)
@@ -7,5 +7,5 @@
     and therefore use a 0.001 mesh scale. Collisions are deliberately simple.
   -->
-  <xacro:macro name="fruit_arm" params="parent hardware_plugin initial_positions_file">
+  <xacro:macro name="fruit_arm" params="parent hardware_plugin initial_positions_file joint_1_rpy joint_2_rpy joint_3_xyz joint_3_rpy joint_4_rpy joint_5_xyz joint_5_rpy joint_6_rpy">
     <xacro:include filename="$(find fruit_arm_moveit_config)/config/fruit_arm.ros2_control.xacro" />
     <xacro:fruit_arm_ros2_control
@@ -53,5 +53,5 @@
     </link>
     <joint name="joint_1" type="revolute">
-      <origin xyz="0 0 0.040975" rpy="0 0 0"/>
+      <origin xyz="0 0 0.040975" rpy="${joint_1_rpy}"/>
       <parent link="cad_base_link"/>
       <child link="arm_link_1"/>
@@ -70,5 +70,5 @@
     <joint name="joint_2" type="revolute">
       <!-- Re-zero CAD assembly angle -65.196838 deg to mechanical J2=0. -->
-      <origin xyz="-0.048101 0.056781 0.094025" rpy="0 -1.137899491 0"/>
+      <origin xyz="-0.048101 0.056781 0.094025" rpy="${joint_2_rpy}"/>
       <parent link="arm_link_1"/>
       <child link="arm_link_2"/>
@@ -89,11 +89,14 @@
     </link>
     <joint name="joint_3" type="revolute">
-      <!-- Re-zero CAD assembly angle +57.956279 deg to perpendicular J3=0. -->
-      <origin xyz="0.399412 -0.015781 0.184581" rpy="0 1.011527890 0"/>
+      <!--
+        Preserve the original drawing-derived installation offset. J3=0 is
+        defined as the horizontal forearm pose by both URDF and controller.
+      -->
+      <origin xyz="${joint_3_xyz}" rpy="${joint_3_rpy}"/>
       <parent link="arm_link_2"/>
       <child link="arm_link_3"/>
       <axis xyz="0 1 0"/>
       <!--
-        Mechanical hard stop: +/-90 deg from perpendicular upper/forearm.
+        Horizontal is 0 deg; the two mechanical hard stops are -90/+90 deg.
       -->
       <limit lower="-1.570796327" upper="1.570796327" effort="180" velocity="1.5"/>
@@ -109,5 +112,5 @@
     <joint name="joint_4" type="revolute">
       <!-- CAD logo-plane reference is opposite mechanical J4 zero. -->
-      <origin xyz="-0.041455 -0.032800 0.057441" rpy="3.141592654 0 0"/>
+      <origin xyz="-0.041455 -0.032800 0.057441" rpy="${joint_4_rpy}"/>
       <parent link="arm_link_3"/>
       <child link="arm_link_4"/>
@@ -126,5 +129,5 @@
     <joint name="joint_5" type="revolute">
       <!-- Re-zero CAD assembly angle +33.439625 deg to mechanical J5=0. -->
-      <origin xyz="-0.372174 -0.034450 -0.004890" rpy="0 0.583631552 0"/>
+      <origin xyz="${joint_5_xyz}" rpy="${joint_5_rpy}"/>
       <parent link="arm_link_4"/>
       <child link="arm_link_5"/>
@@ -144,5 +147,5 @@
     </link>
     <joint name="joint_6" type="revolute">
-      <origin xyz="-0.026883 0.054950 -0.018957" rpy="0 0 0"/>
+      <origin xyz="-0.026883 0.054950 -0.018957" rpy="${joint_6_rpy}"/>
       <parent link="arm_link_5"/>
       <child link="arm_link_6"/>

File: src/moveit_resources-ros2/fruit_arm_moveit_config/config/fruit_picking_arm.urdf.xacro (robot description, xacro)
@@ -7,4 +7,15 @@
   <xacro:arg name="base_xyz" default="0 0 0"/>
   <xacro:arg name="base_rpy" default="0 0 0"/>
+  <!-- Optional per-robot corrections. Defaults reproduce the nominal CAD model. -->
+  <xacro:arg name="joint_1_rpy" default="0 0 0"/>
+  <xacro:arg name="joint_2_rpy" default="0 -1.137899491 0"/>
+  <xacro:arg name="joint_3_xyz" default="0.399412 -0.015781 0.184581"/>
+  <xacro:arg name="joint_3_rpy" default="0 1.011527890 0"/>
+  <xacro:arg name="joint_4_rpy" default="3.141592654 0 0"/>
+  <xacro:arg name="joint_5_xyz" default="-0.372174 -0.034450 -0.004890"/>
+  <xacro:arg name="joint_5_rpy" default="0 0.583631552 0"/>
+  <xacro:arg name="joint_6_rpy" default="0 0 0"/>
+  <xacro:arg name="tcp_xyz" default="0 0 -0.086"/>
+  <xacro:arg name="tcp_rpy" default="0 0 0"/>
   <!--
     Public workcell and robot-base frames.  world owns tables, conveyors,
@@ -27,7 +38,18 @@
       parent="base_link"
       hardware_plugin="$(arg hardware_plugin)"
-      initial_positions_file="$(arg initial_positions_file)" />
+      initial_positions_file="$(arg initial_positions_file)"
+      joint_1_rpy="$(arg joint_1_rpy)"
+      joint_2_rpy="$(arg joint_2_rpy)"
+      joint_3_xyz="$(arg joint_3_xyz)"
+      joint_3_rpy="$(arg joint_3_rpy)"
+      joint_4_rpy="$(arg joint_4_rpy)"
+      joint_5_xyz="$(arg joint_5_xyz)"
+      joint_5_rpy="$(arg joint_5_rpy)"
+      joint_6_rpy="$(arg joint_6_rpy)" />
   <!-- Gripper attached to the arm's tool flange -->
-  <xacro:parallel_jaw_gripper parent="tool_flange" />
+  <xacro:parallel_jaw_gripper
+      parent="tool_flange"
+      tcp_xyz="$(arg tcp_xyz)"
+      tcp_rpy="$(arg tcp_rpy)" />
   <!--
     The fixed eye-to-hand camera is intentionally not part of the robot URDF.

File: src/moveit_resources-ros2/fruit_arm_moveit_config/config/gripper.xacro (robot description, xacro)
@@ -1,5 +1,5 @@
 <?xml version="1.0"?>
 <robot xmlns:xacro="http://www.ros.org/wiki/xacro">
-  <xacro:macro name="parallel_jaw_gripper" params="parent">
+  <xacro:macro name="parallel_jaw_gripper" params="parent tcp_xyz tcp_rpy">
     <!-- Gripper base plate -->
     <link name="gripper_base">
@@ -113,5 +113,5 @@
     <link name="gripper_tcp"/>
     <joint name="gripper_tcp_joint" type="fixed">
-      <origin xyz="0 0 -0.086" rpy="0 0 0"/>
+      <origin xyz="${tcp_xyz}" rpy="${tcp_rpy}"/>
       <parent link="${parent}"/>
       <child link="gripper_tcp"/>

Commit message: Align real arm startup and mechanical joint coordinates

File: src/moveit_resources-ros2/fruit_arm_moveit_config/config/fruit_arm_macro.xacro (robot description, xacro)
@@ -2,8 +2,8 @@
 <robot xmlns:xacro="http://www.ros.org/wiki/xacro">
   <!--
-    Kinematic model inferred from the supplied STEP assembly.  The drawing
-    pose is URDF zero; mechanical reference lines therefore require the
-    documented joint-coordinate offsets below. Visual meshes are millimetres
-    and therefore use a 0.001 mesh scale. Collisions are deliberately simple.
+    Kinematic model derived from the supplied STEP assembly. The mesh assembly
+    pose is converted to the mechanical-zero convention at the joint frames.
+    Visual meshes are millimetres and therefore use a 0.001 mesh scale.
+    Collisions are deliberately simple.
   -->
   <xacro:macro name="fruit_arm" params="parent hardware_plugin initial_positions_file joint_1_rpy joint_2_rpy joint_3_xyz joint_3_rpy joint_4_rpy joint_5_xyz joint_5_rpy joint_6_rpy">
@@ -69,14 +69,14 @@
     </link>
     <joint name="joint_2" type="revolute">
-      <!-- Re-zero CAD assembly angle -65.196838 deg to mechanical J2=0. -->
+      <!--
+        Mechanical J2=0 is the lower hard stop. This is the former model's
+        -60 deg pose re-parameterized as zero: -65.196838 - 60 deg.
+      -->
       <origin xyz="-0.048101 0.056781 0.094025" rpy="${joint_2_rpy}"/>
       <parent link="arm_link_1"/>
       <child link="arm_link_2"/>
       <axis xyz="0 1 0"/>
-      <!--
-        Positive is clockwise when viewed along +Y. Mechanical hard stops:
-        CCW 60 / CW 80 deg.
-      -->
-      <limit lower="-1.047197551" upper="1.396263402" effort="250" velocity="1.5"/>
+      <!-- From the lower hard-stop zero, positive clockwise travel is 144 deg. -->
+      <limit lower="0.0" upper="2.513274123" effort="250" velocity="1.5"/>
     </joint>
     <link name="arm_link_3">
@@ -89,8 +89,5 @@
     </link>
     <joint name="joint_3" type="revolute">
-      <!--
-        Preserve the original drawing-derived installation offset. J3=0 is
-        defined as the horizontal forearm pose by both URDF and controller.
-      -->
+      <!-- Mechanical J3=0 makes the forearm perpendicular to the upper arm. -->
       <origin xyz="${joint_3_xyz}" rpy="${joint_3_rpy}"/>
       <parent link="arm_link_2"/>
@@ -111,11 +108,11 @@
     </link>
     <joint name="joint_4" type="revolute">
-      <!-- CAD logo-plane reference is opposite mechanical J4 zero. -->
+      <!-- Logo shell reference plane defines mechanical J4=0. -->
       <origin xyz="-0.041455 -0.032800 0.057441" rpy="${joint_4_rpy}"/>
       <parent link="arm_link_3"/>
       <child link="arm_link_4"/>
       <axis xyz="1 0 0"/>
-      <!-- Mechanical hard stop: +/-170 deg. -->
-      <limit lower="-2.967059728" upper="2.967059728" effort="120" velocity="1.8"/>
+      <!-- Mechanical hard stop: +/-165 deg. -->
+      <limit lower="-2.879793266" upper="2.879793266" effort="120" velocity="1.8"/>
     </joint>
     <link name="arm_link_5">
@@ -128,5 +125,5 @@
     </link>
     <joint name="joint_5" type="revolute">
-      <!-- Re-zero CAD assembly angle +33.439625 deg to mechanical J5=0. -->
+      <!-- Make the J6 roll axis parallel to the J4 roll axis at mechanical J5=0. -->
       <origin xyz="${joint_5_xyz}" rpy="${joint_5_rpy}"/>
       <parent link="arm_link_4"/>

File: src/moveit_resources-ros2/fruit_arm_moveit_config/config/fruit_picking_arm.urdf.xacro (robot description, xacro)
@@ -7,10 +7,10 @@
   <xacro:arg name="base_xyz" default="0 0 0"/>
   <xacro:arg name="base_rpy" default="0 0 0"/>
-  <!-- Optional per-robot corrections. Defaults reproduce the nominal CAD model. -->
+  <!-- Defaults convert the CAD assembly pose to the currently specified mechanical-zero convention. -->
   <xacro:arg name="joint_1_rpy" default="0 0 0"/>
-  <xacro:arg name="joint_2_rpy" default="0 -1.137899491 0"/>
+  <xacro:arg name="joint_2_rpy" default="0 -2.185097042 0"/>
   <xacro:arg name="joint_3_xyz" default="0.399412 -0.015781 0.184581"/>
-  <xacro:arg name="joint_3_rpy" default="0 1.011527890 0"/>
-  <xacro:arg name="joint_4_rpy" default="3.141592654 0 0"/>
+  <xacro:arg name="joint_3_rpy" default="0 1.137899491 0"/>
+  <xacro:arg name="joint_4_rpy" default="0 0 0"/>
   <xacro:arg name="joint_5_xyz" default="-0.372174 -0.034450 -0.004890"/>
   <xacro:arg name="joint_5_rpy" default="0 0.583631552 0"/>
